File: kicad/cpu6809.sch (KiCad schematic (older format))
At the start: 24 parts, among them J1 Conn_01x02_Male, Q1 3.6864Mhz, SW1 SW_Push, U1 TL7705A, U2 MC6809, U3 GAL22V10, U4 74LS138

Commit message: Adding PCB layout
Parts:
- removed C27: 47u/16V, Capacitors_THT:CP_Radial_D5.0mm_P2.50mm, symbol Device:CP
- removed R2, R3, R4, R5, R6, R7, R8: 4k7, symbol Device:R
- added J6: Conn_01x03_Male, Connectors_Molex:Molex_KK-6410-03_03x2.54mm_Straight, symbol Connector:Conn_01x03_Male
- added J7: Conn_01x02_Male, Connectors_Molex:Molex_KK-6410-02_02x2.54mm_Straight, symbol Connector:Conn_01x02_Male
- added J8: Conn_01x02_Male, Pin_Headers:Pin_Header_Straight_1x02_Pitch2.54mm, symbol Connector:Conn_01x02_Male
- added RN1: 4k7, Resistors_THT:R_Array_SIP8, symbol Device:R_Network07
- added TP1: E, Connectors:Pin_d1.0mm_L10.0mm, symbol Connector:TestPoint
- added TP2: GND, Connectors:Pin_d1.0mm_L10.0mm, symbol Connector:TestPoint
- added TP5: +5V, Connectors:Pin_d1.0mm_L10.0mm, symbol Connector:TestPoint
- J1: footprint (none) -> Connectors:JACK_ALIM
- Q1: footprint (none) -> Crystals:Crystal_HC18-U_Vertical
- SW1: footprint (none) -> Buttons_Switches_THT:SW_PUSH_6mm
- U4: footprint Housings_DIP:DIP-8_W7.62mm_Socket_LongPads -> Housings_DIP:DIP-16_W7.62mm_LongPads
Connections:
- net labels added: BA, BS, Q, ~DMA~, ~HALT~, ~MRDY~
- wire segments 158 -> 176
Other:
- moved on the sheet: C5
