File: kicad/mc6809.sch (KiCad schematic (older format))
At the start: 0 parts

Commit message: Adding PCB layout
Changed lines of the file:
@@
 $Descr A4 11693 8268
 encoding utf-8
-Sheet 1 6
+Sheet 1 7
 Title ""
 Date ""
@@
 F1 "floppy.sch" 50
 $EndSheet
+$Sheet
+S 1600 3000 1250 850
+U 612261E0
+F0 "ext" 50
+F1 "ext.sch" 50
+$EndSheet
 $EndSCHEMATC
