File: kicad/mem.sch (KiCad schematic (older format))
At the start: 6 parts, among them U10 MK48T12, U8 27C64, U9 628128_DIP32_SSOP32

Commit message: Adding PCB layout
Parts:
- U10: footprint (none) -> Housings_DIP:DIP-24_W15.24mm_LongPads
Changed lines of the file:
@@
 $Descr A4 11693 8268
 encoding utf-8
-Sheet 4 6
+Sheet 4 7
 Title ""
 Date ""
@@
 F 0 "U10" H 2450 4100 50  0000 C CNN
 F 1 "MK48T12" H 2600 4000 50  0000 C CNN
-F 2 "" H 2300 2850 50  0001 C CNN
+F 2 "Housings_DIP:DIP-24_W15.24mm_LongPads" H 2300 2850 50  0001 C CNN
 F 3 "" H 2300 2850 50  0001 C CNN
 	1    2300 2850
@@
 ~CSRTC~
 Text GLabel 2550 6700 2    50   UnSpc ~ 0
-~WR~
+~CSRAM~
 Text GLabel 2550 6850 2    50   UnSpc ~ 0
 ~CSROM~
