File: kicad/ext.sch (KiCad schematic (older format))
At the start: 1 part, among them J5 DIN41612-a+c

Commit message: Adding PCB
Parts:
- J5: footprint mylib:Socket_DIN41612-CaseC1-AC-Male-64Pin-2rows -> mylib:Socket_DIN41612-CaseC1-AC-Male-64Pin-2rows-nosilk
Changed lines of the file:
@@
 F 0 "J5" H 5900 4717 50  0000 C CNN
 F 1 "DIN41612-a+c" H 5900 4626 50  0000 C CNN
-F 2 "mylib:Socket_DIN41612-CaseC1-AC-Male-64Pin-2rows" H 5850 3000 50  0001 C CNN
+F 2 "mylib:Socket_DIN41612-CaseC1-AC-Male-64Pin-2rows-nosilk" H 5850 3000 50  0001 C CNN
 F 3 "~" H 5850 3000 50  0001 C CNN
 	1    5850 3000
